Commit message: update gazebo working now with reduced files

File: baxter/baxter_common/baxter_description/urdf/baxter.urdf.xacro (robot description, xacro)
@@ -1,7 +1,6 @@
 <?xml version="1.0" ?>
 <robot name="baxter" xmlns:xacro="http://www.ros.org/wiki/xacro">
-  <xacro:arg name="gazebo" default="true"/>
+  <xacro:arg name="gazebo" default="false"/>
   <xacro:arg name="pedestal" default="true"/>
-  <xacro:arg name="coffe_table" default="true"/>
   <!-- Baxter Base URDF -->
   <xacro:include filename="$(find baxter_description)/urdf/baxter_base/baxter_base.urdf.xacro">
@@ -18,10 +17,3 @@
   <!-- Right End Effector -->
   <xacro:include filename="$(find baxter_description)/urdf/right_end_effector.urdf.xacro" />
-  <!-- Coffe Table -->
-  <!-- <xacro:include filename="$(find baxter_sim_examples)/models/cafe_table/model.xacro" /> -->
-  <!-- Kinect Sensor -->
- <!-- <xacro:if value="$(arg gazebo)">
-    <xacro:include filename="$(find baxter_description)/urdf/depth_sensor.urdf.xacro" />
-    <sensor_kinect parent="base" location="1.0 -0.0125 2.0" orientation="0 1.57 0.0"/>
-  </xacro:if> -->
 </robot>

File: baxter/baxter_common/baxter_description/urdf/baxter_base/baxter_base.gazebo.xacro (robot description, xacro)
@@ -5,11 +5,9 @@
     <plugin name="baxter_ros_control" filename="libbaxter_gazebo_ros_control.so">
       <robotNamespace>/robot</robotNamespace>
-      <robotSimType>gazebo_ros_control/DefaultRobotHWSim</robotSimType> <!-- Gazebo Default -->
-      <controlPeriod>0.001</controlPeriod> <!-- Gazebo Default -->
     </plugin>
   </gazebo>
   <!-- Gazebo-Specific Link Properties -->
   <gazebo reference="torso">
-    <self_collide>true</self_collide>
+    <selfCollide>true</selfCollide>
   </gazebo>
   <gazebo reference="head_pan">
@@ -93,8 +91,4 @@
         <distortionT1>0.0</distortionT1>
         <distortionT2>0.0</distortionT2>
-        <CxPrime>0</CxPrime>
-        <Cx>0.0</Cx>
-        <Cy>0.0</Cy>
-        <focalLength>0.0</focalLength>
         <robotNamespace>/cameras</robotNamespace>
       </plugin>
@@ -135,8 +129,4 @@
         <distortionT1>0.0</distortionT1>
         <distortionT2>0.0</distortionT2>
-        <CxPrime>0</CxPrime>
-        <Cx>0.0</Cx>
-        <Cy>0.0</Cy>
-        <focalLength>0.0</focalLength>
         <robotNamespace>/cameras</robotNamespace>
       </plugin>
@@ -177,8 +167,4 @@
         <distortionT1>0.0</distortionT1>
         <distortionT2>0.0</distortionT2>
-        <CxPrime>0</CxPrime>
-        <Cx>0.0</Cx>
-        <Cy>0.0</Cy>
-        <focalLength>0.0</focalLength>
         <robotNamespace>/cameras</robotNamespace>
       </plugin>
@@ -191,5 +177,4 @@
         <width>1024</width>
         <topicName>/robot/xdisplay</topicName>
-        <robotNamespace>/robot</robotNamespace>
       </plugin>
     </visual>
@@ -224,5 +209,4 @@
         <topicName>/robot/sonar/head_sonar/state</topicName>
         <frameName>sonar_ring</frameName>
-        <hokuyoMinIntensity>101</hokuyoMinIntensity>
       </plugin>
       <always_on>true</always_on>
@@ -291,8 +275,8 @@
     <type>transmission_interface/SimpleTransmission</type>
     <joint name="right_s0">
-      <hardwareInterface>hardware_interface/EffortJointInterface</hardwareInterface>
+      <hardwareInterface>EffortJointInterface</hardwareInterface>
     </joint>
     <actuator name="right_motor1">
-      <hardwareInterface>hardware_interface/EffortJointInterface</hardwareInterface>
+      <hardwareInterface>EffortJointInterface</hardwareInterface>
       <mechanicalReduction>1</mechanicalReduction>
     </actuator>
@@ -301,8 +285,8 @@
     <type>transmission_interface/SimpleTransmission</type>
     <joint name="right_s1">
-      <hardwareInterface>hardware_interface/EffortJointInterface</hardwareInterface>
+      <hardwareInterface>EffortJointInterface</hardwareInterface>
     </joint>
     <actuator name="right_motor2">
-      <hardwareInterface>hardware_interface/EffortJointInterface</hardwareInterface>
+      <hardwareInterface>EffortJointInterface</hardwareInterface>
       <mechanicalReduction>1</mechanicalReduction>
     </actuator>
@@ -311,8 +295,8 @@
     <type>transmission_interface/SimpleTransmission</type>
     <joint name="right_e0">
-      <hardwareInterface>hardware_interface/EffortJointInterface</hardwareInterface>
+      <hardwareInterface>EffortJointInterface</hardwareInterface>
     </joint>
     <actuator name="right_motor3">
-      <hardwareInterface>hardware_interface/EffortJointInterface</hardwareInterface>
+      <hardwareInterface>EffortJointInterface</hardwareInterface>
       <mechanicalReduction>1</mechanicalReduction>
     </actuator>
@@ -321,8 +305,8 @@
     <type>transmission_interface/SimpleTransmission</type>
     <joint name="right_e1">
-      <hardwareInterface>hardware_interface/EffortJointInterface</hardwareInterface>
+      <hardwareInterface>EffortJointInterface</hardwareInterface>
     </joint>
     <actuator name="right_motor4">
-      <hardwareInterface>hardware_interface/EffortJointInterface</hardwareInterface>
+      <hardwareInterface>EffortJointInterface</hardwareInterface>
       <mechanicalReduction>1</mechanicalReduction>
     </actuator>
@@ -331,8 +315,8 @@
     <type>transmission_interface/SimpleTransmission</type>
     <joint name="right_w0">
-      <hardwareInterface>hardware_interface/EffortJointInterface</hardwareInterface>
+      <hardwareInterface>EffortJointInterface</hardwareInterface>
     </joint>
     <actuator name="right_motor5">
-      <hardwareInterface>hardware_interface/EffortJointInterface</hardwareInterface>
+      <hardwareInterface>EffortJointInterface</hardwareInterface>
       <mechanicalReduction>1</mechanicalReduction>
     </actuator>
@@ -341,8 +325,8 @@
     <type>transmission_interface/SimpleTransmission</type>
     <joint name="right_w1">
-      <hardwareInterface>hardware_interface/EffortJointInterface</hardwareInterface>
+      <hardwareInterface>EffortJointInterface</hardwareInterface>
     </joint>
     <actuator name="right_motor6">
-      <hardwareInterface>hardware_interface/EffortJointInterface</hardwareInterface>
+      <hardwareInterface>EffortJointInterface</hardwareInterface>
       <mechanicalReduction>1</mechanicalReduction>
     </actuator>
@@ -351,8 +335,8 @@
     <type>transmission_interface/SimpleTransmission</type>
     <joint name="right_w2">
-      <hardwareInterface>hardware_interface/EffortJointInterface</hardwareInterface>
+      <hardwareInterface>EffortJointInterface</hardwareInterface>
     </joint>
     <actuator name="right_motor7">
-      <hardwareInterface>hardware_interface/EffortJointInterface</hardwareInterface>
+      <hardwareInterface>EffortJointInterface</hardwareInterface>
       <mechanicalReduction>1</mechanicalReduction>
     </actuator>
@@ -362,8 +346,8 @@
     <type>transmission_interface/SimpleTransmission</type>
     <joint name="left_s0">
-      <hardwareInterface>hardware_interface/EffortJointInterface</hardwareInterface>
+      <hardwareInterface>EffortJointInterface</hardwareInterface>
     </joint>
     <actuator name="left_motor1">
-      <hardwareInterface>hardware_interface/EffortJointInterface</hardwareInterface>
+      <hardwareInterface>EffortJointInterface</hardwareInterface>
       <mechanicalReduction>1</mechanicalReduction>
     </actuator>
@@ -372,8 +356,8 @@
     <type>transmission_interface/SimpleTransmission</type>
     <joint name="left_s1">
-      <hardwareInterface>hardware_interface/EffortJointInterface</hardwareInterface>
+      <hardwareInterface>EffortJointInterface</hardwareInterface>
     </joint>
     <actuator name="left_motor2">
-      <hardwareInterface>hardware_interface/EffortJointInterface</hardwareInterface>
+      <hardwareInterface>EffortJointInterface</hardwareInterface>
       <mechanicalReduction>1</mechanicalReduction>
     </actuator>
@@ -382,8 +366,8 @@
     <type>transmission_interface/SimpleTransmission</type>
     <joint name="left_e0">
-      <hardwareInterface>hardware_interface/EffortJointInterface</hardwareInterface>
+      <hardwareInterface>EffortJointInterface</hardwareInterface>
     </joint>
     <actuator name="left_motor3">
-      <hardwareInterface>hardware_interface/EffortJointInterface</hardwareInterface>
+      <hardwareInterface>EffortJointInterface</hardwareInterface>
       <mechanicalReduction>1</mechanicalReduction>
     </actuator>
@@ -392,8 +376,8 @@
     <type>transmission_interface/SimpleTransmission</type>
     <joint name="left_e1">
-      <hardwareInterface>hardware_interface/EffortJointInterface</hardwareInterface>
+      <hardwareInterface>EffortJointInterface</hardwareInterface>
     </joint>
     <actuator name="left_motor4">
-      <hardwareInterface>hardware_interface/EffortJointInterface</hardwareInterface>
+      <hardwareInterface>EffortJointInterface</hardwareInterface>
       <mechanicalReduction>1</mechanicalReduction>
     </actuator>
@@ -402,8 +386,8 @@
     <type>transmission_interface/SimpleTransmission</type>
     <joint name="left_w0">
-      <hardwareInterface>hardware_interface/EffortJointInterface</hardwareInterface>
+      <hardwareInterface>EffortJointInterface</hardwareInterface>
     </joint>
     <actuator name="left_motor5">
-      <hardwareInterface>hardware_interface/EffortJointInterface</hardwareInterface>
+      <hardwareInterface>EffortJointInterface</hardwareInterface>
       <mechanicalReduction>1</mechanicalReduction>
     </actuator>
@@ -412,8 +396,8 @@
     <type>transmission_interface/SimpleTransmission</type>
     <joint name="left_w1">
-      <hardwareInterface>hardware_interface/EffortJointInterface</hardwareInterface>
+      <hardwareInterface>EffortJointInterface</hardwareInterface>
     </joint>
     <actuator name="left_motor6">
-      <hardwareInterface>hardware_interface/EffortJointInterface</hardwareInterface>
+      <hardwareInterface>EffortJointInterface</hardwareInterface>
       <mechanicalReduction>1</mechanicalReduction>
     </actuator>
@@ -422,8 +406,8 @@
     <type>transmission_interface/SimpleTransmission</type>
     <joint name="left_w2">
-      <hardwareInterface>hardware_interface/EffortJointInterface</hardwareInterface>
+      <hardwareInterface>EffortJointInterface</hardwareInterface>
     </joint>
     <actuator name="left_motor7">
-      <hardwareInterface>hardware_interface/EffortJointInterface</hardwareInterface>
+      <hardwareInterface>EffortJointInterface</hardwareInterface>
       <mechanicalReduction>1</mechanicalReduction>
     </actuator>
@@ -433,8 +417,8 @@
     <type>transmission_interface/SimpleTransmission</type>
     <joint name="head_pan">
-      <hardwareInterface>hardware_interface/EffortJointInterface</hardwareInterface>
+      <hardwareInterface>EffortJointInterface</hardwareInterface>
     </joint>
     <actuator name="head_motor1">
-      <hardwareInterface>hardware_interface/EffortJointInterface</hardwareInterface>
+      <hardwareInterface>EffortJointInterface</hardwareInterface>
       <mechanicalReduction>1</mechanicalReduction>
     </actuator>

File: baxter/baxter_common/baxter_description/urdf/baxter_base/baxter_base.urdf.xacro (robot description, xacro)
@@ -12,5 +12,5 @@
       <origin rpy="0 0 0" xyz="0 0 0"/>
       <geometry>
-        <mesh filename="package://$(find baxter_description)/meshes/torso/base_link.DAE"/>
+        <mesh filename="package://baxter_description/meshes/torso/base_link.DAE"/>
       </geometry>
       <material name="darkgray">
@@ -21,5 +21,5 @@
       <origin rpy="0 0 0" xyz="0 0 0"/>
       <geometry>
-        <mesh filename="package://$(find baxter_description)/meshes/torso/base_link_collision.DAE"/>
+        <mesh filename="package://baxter_description/meshes/torso/base_link_collision.DAE"/>
       </geometry>
     </collision>
@@ -92,5 +92,5 @@
       <origin rpy="0 -1.57079632679 0" xyz="0 -.00953 -.0347"/>
       <geometry>
-        <mesh filename="package://$(find baxter_description)/meshes/head/H1.DAE"/>
+        <mesh filename="package://baxter_description/meshes/head/H1.DAE"/>
       </geometry>
       <material name="darkred">
@@ -186,10 +186,10 @@
   <joint name="collision_head_1" type="fixed">
     <origin rpy="0 0 0" xyz="0.11 0 0.75"/>
-    <parent link="torso"/>
+    <parent link="base"/>
     <child link="collision_head_link_1"/>
   </joint>
   <joint name="collision_head_2" type="fixed">
     <origin rpy="0 0 0" xyz="0.11 0 0.75"/>
-    <parent link="torso"/>
+    <parent link="base"/>
     <child link="collision_head_link_2"/>
   </joint>
@@ -200,5 +200,5 @@
   </joint>
   <joint name="torso_t0" type="fixed">
-    <origin rpy="0 0 0" xyz="0 0 0.93"/>
+    <origin rpy="0 0 0" xyz="0 0 0"/>
     <parent link="base"/>
     <child link="torso"/>
@@ -256,5 +256,5 @@
       <origin rpy="0 0 0" xyz="0 0 0"/>
       <geometry>
-        <mesh filename="package://$(find baxter_description)/meshes/upper_shoulder/S0.DAE"/>
+        <mesh filename="package://baxter_description/meshes/upper_shoulder/S0.DAE"/>
       </geometry>
       <material name="darkred">
@@ -278,5 +278,5 @@
       <origin rpy="0 0 0" xyz="0 0 0"/>
       <geometry>
-        <mesh filename="package://$(find baxter_description)/meshes/lower_shoulder/S1.DAE"/>
+        <mesh filename="package://baxter_description/meshes/lower_shoulder/S1.DAE"/>
       </geometry>
       <material name="darkred">
@@ -300,5 +300,5 @@
       <origin rpy="0 0 0" xyz="0 0 0"/>
       <geometry>
-        <mesh filename="package://$(find baxter_description)/meshes/upper_elbow/E0.DAE"/>
+        <mesh filename="package://baxter_description/meshes/upper_elbow/E0.DAE"/>
       </geometry>
       <material name="darkred">
@@ -335,5 +335,5 @@
       <origin rpy="0 0 0" xyz="0 0 0"/>
       <geometry>
-        <mesh filename="package://$(find baxter_description)/meshes/lower_elbow/E1.DAE"/>
+        <mesh filename="package://baxter_description/meshes/lower_elbow/E1.DAE"/>
       </geometry>
       <material name="darkred">
@@ -357,5 +357,5 @@
       <origin rpy="0 0 0" xyz="0 0 0"/>
       <geometry>
-        <mesh filename="package://$(find baxter_description)/meshes/upper_forearm/W0.DAE"/>
+        <mesh filename="package://baxter_description/meshes/upper_forearm/W0.DAE"/>
       </geometry>
       <material name="darkred">
@@ -399,5 +399,5 @@
       <origin rpy="0 0 0" xyz="0 0 0"/>
       <geometry>
-        <mesh filename="package://$(find baxter_description)/meshes/lower_forearm/W1.DAE"/>
+        <mesh filename="package://baxter_description/meshes/lower_forearm/W1.DAE"/>
       </geometry>
       <material name="darkred">
@@ -421,5 +421,5 @@
       <origin rpy="0 0 0" xyz="0 0 0"/>
       <geometry>
-        <mesh filename="package://$(find baxter_description)/meshes/wrist/W2.DAE"/>
+        <mesh filename="package://baxter_description/meshes/wrist/W2.DAE"/>
       </geometry>
       <material name="lightgrey">
@@ -624,5 +624,5 @@
       <origin rpy="0 0 0" xyz="0 0 0"/>
       <geometry>
-        <mesh filename="package://$(find baxter_description)/meshes/upper_shoulder/S0.DAE"/>
+        <mesh filename="package://baxter_description/meshes/upper_shoulder/S0.DAE"/>
       </geometry>
       <material name="darkred">
@@ -646,5 +646,5 @@
       <origin rpy="0 0 0" xyz="0 0 0"/>
       <geometry>
-        <mesh filename="package://$(find baxter_description)/meshes/lower_shoulder/S1.DAE"/>
+        <mesh filename="package://baxter_description/meshes/lower_shoulder/S1.DAE"/>
       </geometry>
       <material name="darkred">
@@ -668,5 +668,5 @@
       <origin rpy="0 0 0" xyz="0 0 0"/>
       <geometry>
-        <mesh filename="package://$(find baxter_description)/meshes/upper_elbow/E0.DAE"/>
+        <mesh filename="package://baxter_description/meshes/upper_elbow/E0.DAE"/>
       </geometry>
       <material name="darkred">
@@ -703,5 +703,5 @@
       <origin rpy="0 0 0" xyz="0 0 0"/>
       <geometry>
-        <mesh filename="package://$(find baxter_description)/meshes/lower_elbow/E1.DAE"/>
+        <mesh filename="package://baxter_description/meshes/lower_elbow/E1.DAE"/>
       </geometry>
       <material name="darkred">
@@ -725,5 +725,5 @@
       <origin rpy="0 0 0" xyz="0 0 0"/>
       <geometry>
-        <mesh filename="package://$(find baxter_description)/meshes/upper_forearm/W0.DAE"/>
+        <mesh filename="package://baxter_description/meshes/upper_forearm/W0.DAE"/>
       </geometry>
       <material name="darkred">
@@ -767,5 +767,5 @@
       <origin rpy="0 0 0" xyz="0 0 0"/>
       <geometry>
-        <mesh filename="package://$(find baxter_description)/meshes/lower_forearm/W1.DAE"/>
+        <mesh filename="package://baxter_description/meshes/lower_forearm/W1.DAE"/>
       </geometry>
       <material name="darkred">
@@ -789,5 +789,5 @@
       <origin rpy="0 0 0" xyz="0 0 0"/>
       <geometry>
-        <mesh filename="package://$(find baxter_description)/meshes/wrist/W2.DAE"/>
+        <mesh filename="package://baxter_description/meshes/wrist/W2.DAE"/>
       </geometry>
       <material name="lightgrey">
